File: schematics/Bosch eBike Charger BCS220/Bosch eBike Charger BCS220.kicad_sch (KiCad schematic)
At the start: 93 parts, among them J1 Netz, Q2 SVF13N50T, Q5 SVF13N50T, Q8 MJE13003, U2 L6599, U6 20J25

Commit message: - update gitignore files
- some cleanups in schematics
Parts:
- added C42: (no value), symbol Device:C_Small
- added C44: (no value), symbol Device:C_Polarized_Small
- added D12: (no value), symbol Device:D
- added R70: 47R, symbol Device:R
- added R76: 2k, symbol Device:R
- added R86: 2R2, symbol Device:R
- R15, R44: value (none) -> 47
- R40: value 1,87k -> 1.87k
- R51, R9: value (none) -> 100k
Connections:
- net TR5_4 is gone; now on net GND: C2.2, TR5.4 (SB)
- net U3_C: now also R40.1; no longer R40.2
- net U7_C: now also R100.1; no longer R100.2
- net at R31.1, R47.1, U2.4 (RFMIN): now also R40.2; no longer R40.1
- net at C1.1, U6.1 (Phase): now also R83.1; no longer R83.2
- net at R82.1, TR2.6 (SD): now also R104.2; no longer R104.1
- net at D14.2 (A): now also R104.1; no longer R104.2
- net at Q12.1 (B), R105.2: now also R100.2; no longer R100.1
- net at R82.2, R84.1: now also R83.2; no longer R83.1
- net T2_3: no longer names the net of TR2.3 (SA)
- net T2_3: now also D12.2 (A), R70.1
- net T2_4 renamed GND
- net GND: now also C44.2, R76.2
- net primPlusFilt: no longer names the net of C46.1, L5.2, R73.1, R74.1, R75.1, R99.2, TR2.1 (AA)
- new net: C42.1, R70.2
- new net V+: R86.2
- new net VSup+: C42.2, C44.1, D12.1 (K), R76.1, R86.1
Other:
- note added: "Charge Control Input"
- moved on the sheet: C1, C10, C14, C16, C17, C18, C2, C20, C21, C26, C28, C29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
