File: schematics/Bosch eBike Charger BCS220/secondary1.kicad_sch (KiCad schematic)
At the start: 70 parts, among them K1 Relay_SPST-NO, Q17 2N7002, Q18 2N3904, Q4 AFT3904, Q6 AFT3904, Q7 AFT3904, U1 LM324, U3 LTV-817, U5 WL431, U8 WL431, U9 WL431

Commit message: - update gitignore files
- some cleanups in schematics
Parts:
- removed C42: (no value), symbol Device:C_Small
- removed C44: (no value), symbol Device:C_Polarized_Small
- removed D12: (no value), symbol Device:D
- removed R70: 47R, symbol Device:R
- removed R76: 2k, symbol Device:R
- removed R86: 2R2, symbol Device:R
Connections:
- net +5V: now also R149.2; no longer R149.1
- net GND: now also C57.2, C74.2, C75.2, C80.2, C84.2, C86.1, L1.1 (AA), Q17.2 (S), Q4.2 (E), R146.2, R202.2, R33.2, R81.2, U5.3 (A), U9.3 (A)
- net at C84.1, L8.1, R139.2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: now also R149.1; no longer R149.2
Other:
- moved on the sheet: C74, C75, C81, C84, L8, Q18, R139, R145, R146, R147, R149, R201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
